Commit message: Update base.urdf.xacro to include 2 connections on base_footprint

File: omni_base_description/urdf/base/base.urdf.xacro (robot description, xacro)
@@ -68,4 +68,16 @@
       <parent link="${name}_footprint"/>
     </joint>
+    <link name="${name}_connection"/>
+    <joint name="${name}_connection_joint" type="fixed">
+      <origin xyz="0 0.08 0" rpy="0 0 0" />
+      <child link="${name}_footprint" />
+      <parent link="${name}_connection"/>
+    </joint>
+    <link name="${name}_connection2"/>
+    <joint name="${name}_connection_joint2" type="fixed">
+      <origin xyz="0 -0.08 0" rpy="0 0 0" />
+      <child link="${name}_footprint" />
+      <parent link="${name}_connection2"/>
+    </joint>
   <!-- gazebo parameters are given here for base_link through base_footprint -->
     <gazebo reference="${name}_footprint">
